Commit message: updated Files to Work in Gazebo and RVIZ

File: src/robot_sim/urdf/watcher.urdf.xacro (robot description, xacro)
@@ -20,4 +20,10 @@
             </geometry>
         </collision>
+    <!--Added inertial tags HERE-->
+        <inertial>
+            <mass value="15.0"/>
+            <origin xyz="0 0 0.1778" rpy="0 0 0"/>
+            <inertia ixx="0.2" ixy="0.0" ixz="0.0" iyy="0.2" iyz="0.0" izz="0.2"/>
+        </inertial>
     </link>
     <joint name="right_wheel_joint" type="continuous">
@@ -40,4 +46,10 @@
             </geometry>
         </collision>
+    <!--Added interial tags HERE-->
+        <inertial>
+            <mass value="2.0"/>
+            <origin xyz="0 0 0" rpy="0 0 0"/>
+            <inertia ixx="0.01" ixy="0.0" ixz="0.0" iyy="0.01" iyz="0.0" izz="0.01"/>
+        </inertial>
     </link>
     <joint name="left_wheel_joint" type="continuous">
@@ -60,4 +72,10 @@
             </geometry>
         </collision>
+        <!--Added interial tags HERE-->
+        <inertial>
+            <mass value="2.0"/>
+            <origin xyz="0 0 0" rpy="0 0 0"/>
+            <inertia ixx="0.01" ixy="0.0" ixz="0.0" iyy="0.01" iyz="0.0" izz="0.01"/>
+        </inertial>
     </link>
     <joint name="chair_joint" type="fixed">
@@ -79,4 +97,10 @@
             </geometry>
         </collision>
+        <!--Added interial tags HERE-->
+        <inertial>
+            <mass value="10.0"/>
+            <origin xyz="0 0 0.3556" rpy="0 0 0"/>
+            <inertia ixx="0.3" ixy="0.0" ixz="0.0" iyy="0.3" iyz="0.0" izz="0.3"/>
+        </inertial>
     </link>
 </robot>

Commit message: Changed model and added Depth Camera

File: src/robot_sim/urdf/watcher.urdf.xacro (robot description, xacro)
@@ -5,31 +5,33 @@
         <parent link="base_footprint"/>
         <child link="base_link"/>
-        <origin rpy="0 0 0" xyz="0 0 0.05"/>
-    </joint>
+        <origin rpy="0 0 0" xyz="0 0 0.0"/>
+    </joint>
+    <!--Motor BASE-->
     <link name="base_link">
         <visual>
             <origin rpy="0 0 0" xyz="0 0 0.1778"/>
             <geometry>
+                <box size="0.6096 0.4953 0.3556"/> <!--24x19.5x14 inches-->
+            </geometry>
+        </visual>
+        <collision>
+            <origin rpy="0 0 0" xyz="0 0 0.1778"/>
+            <geometry>
                 <box size="0.6096 0.4953 0.3556"/>
             </geometry>
-        </visual>
-        <collision>
-            <origin rpy="0 0 0" xyz="0 0 0.1778"/>
-            <geometry>
-                <box size="0.6096 0.4953 0.3556"/>
-            </geometry>
         </collision>
     <!--Added inertial tags HERE-->
         <inertial>
-            <mass value="15.0"/>
+            <mass value="30.0"/>
             <origin xyz="0 0 0.1778" rpy="0 0 0"/>
-            <inertia ixx="0.2" ixy="0.0" ixz="0.0" iyy="0.2" iyz="0.0" izz="0.2"/>
-        </inertial>
-    </link>
+            <inertia ixx="1.0" ixy="0.0" ixz="0.0" iyy="1.0" iyz="0.0" izz="1.0"/>
+        </inertial>
+    </link>
+    <!--DRIVE WHEELS-->
     <joint name="right_wheel_joint" type="continuous">
         <parent link="base_link"/>
         <child link="right_wheel"/>
         <axis xyz="0 1 0"/>
-        <origin rpy="0 0 0" xyz="0 -0.2794 0.1778"/>
+        <origin rpy="0 0 0" xyz="0 0.24765 0.15875"/>
     </joint>
     <link name="right_wheel">
@@ -37,5 +39,5 @@
             <origin rpy="1.5708 0 0" xyz="0 0 0"/>
             <geometry>
-                <cylinder radius="0.3175" length="0.0508"/>
+                <cylinder radius="0.15875" length="0.0508"/>
             </geometry>
         </visual>
@@ -43,6 +45,17 @@
             <origin rpy="1.5708 0 0" xyz="0 0 0"/>
             <geometry>
-                <cylinder radius="0.3175" length="0.0508"/>
-            </geometry>
+                <cylinder radius="0.15875" length="0.0508"/>
+            </geometry>
+            <surface>
+                <contact>
+                    <ode/>
+                </contact>
+            <friction>
+                <ode>
+                <mu>2.0</mu>
+                <mu2>2.0</mu2>
+                </ode>
+            </friction>
+        </surface>
         </collision>
     <!--Added interial tags HERE-->
@@ -53,9 +66,14 @@
         </inertial>
     </link>
+    <!--Friction Right wheel-->
+    <gazebo reference="right_wheel">
+        <mu1>2.0</mu1>
+        <mu2>2.0</mu2>
+    </gazebo>
     <joint name="left_wheel_joint" type="continuous">
         <parent link="base_link"/>
         <child link="left_wheel"/>
         <axis xyz="0 1 0"/>
-        <origin rpy="0 0 0" xyz="0 0.2794 0.1778"/>
+        <origin rpy="0 0 0" xyz="0 -0.24765 0.15875"/>
     </joint>
     <link name="left_wheel">
@@ -63,5 +81,5 @@
             <origin rpy="1.5708 0 0" xyz="0 0 0"/>
             <geometry>
-                <cylinder radius="0.3175" length="0.0508"/>
+                <cylinder radius="0.15875" length="0.0508"/>
             </geometry>
         </visual>
@@ -69,6 +87,17 @@
             <origin rpy="1.5708 0 0" xyz="0 0 0"/>
             <geometry>
-                <cylinder radius="0.3175" length="0.0508"/>
-            </geometry>
+                <cylinder radius="0.15875" length="0.0508"/>
+            </geometry>
+            <surface>
+                <contact>
+                    <ode/>
+                </contact>
+            <friction>
+                <ode>
+                <mu>2.0</mu>
+                <mu2>2.0</mu2>
+                </ode>
+            </friction>
+        </surface>
         </collision>
         <!--Added interial tags HERE-->
@@ -79,8 +108,146 @@
         </inertial>
     </link>
+    <!--Friction For Left wheels -->
+    <gazebo reference="left_wheel">
+        <mu1>2.0</mu1>
+        <mu2>2.0</mu2>
+    </gazebo>
+    <!--Front left Caster Wheel-->
+    <joint name="front_left_caster_joint" type="revolute">
+        <parent link="base_link"/>
+        <child link="front_left_caster"/>
+        <origin xyz="0.3429 0.24765 0.0762" rpy="0 0 0"/>
+        <axis  xyz = "0 0 1"/>
+        <limit effort = "1.0" velocity = "5.0" lower ="-3.14" upper = "3.14" />
+        <dynamics damping = "0.2"/>
+    </joint>
+    <link name="front_left_caster">
+        <visual>
+            <origin xyz="0 0 0" rpy="1.5708 0 0"/>
+            <geometry>
+                <cylinder radius="0.0762" length="0.0508"/>
+            </geometry>
+        </visual>
+        <collision>
+            <origin xyz="0 0 0" rpy="1.5708 0 0"/>
+            <geometry>
+                <cylinder radius="0.0762" length="0.0508"/>
+            </geometry>
+        </collision>
+        <inertial>
+            <mass value="0.5"/>
+            <origin xyz="0 0 0" rpy="0 0 0"/>
+            <inertia ixx="0.001" iyy="0.001" izz="0.001" ixy="0.0" ixz="0.0" iyz="0.0"/>
+        </inertial>
+    </link>
+    <!--Friction for Left Caster wheel-->
+    <gazebo reference="front_left_caster">
+        <mu1>0.01</mu1>
+        <mu2>0.01</mu2>
+    </gazebo>
+    <!--Front Right Caster Wheel-->
+    <joint name="front_right_caster_joint" type="revolute">
+        <parent link="base_link"/>
+        <child link="front_right_caster"/>
+        <origin xyz="0.3429 -0.24765 0.0762" rpy="0 0 0"/>
+        <axis xyz = "0 0 1"/>
+        <limit effort = "1.0" velocity = "5.0" lower ="-3.14" upper = "3.14" />
+        <dynamics damping = "0.2"/>
+    </joint>
+    <link name="front_right_caster">
+        <visual>
+            <origin xyz="0 0 0" rpy="1.5708 0 0"/>
+            <geometry>
+                <cylinder radius="0.0762" length="0.0508"/>
+            </geometry>
+        </visual>
+        <collision>
+            <origin xyz="0 0 0" rpy="1.5708 0 0"/>
+            <geometry>
+                <cylinder radius="0.0762" length="0.0508"/>
+            </geometry>
+        </collision>
+        <inertial>
+            <mass value="0.5"/>
+            <origin xyz="0 0 0" rpy="0 0 0"/>
+            <inertia ixx="0.001" iyy="0.001" izz="0.001" ixy="0.0" ixz="0.0" iyz="0.0"/>
+        </inertial>
+    </link>
+    <!--Friction for front right Caster-->
+    <gazebo reference="front_right_caster">
+        <mu1>0.1</mu1>
+        <mu2>0.1</mu2>
+    </gazebo>
+    <!--Rear Left  Caster Wheel-->
+    <joint name="rear_left_caster_joint" type="revolute">
+        <parent link="base_link"/>
+        <child link="rear_left_caster"/>
+        <origin xyz="-0.4699 0.24765 0.0762" rpy="0 0 0"/>
+        <axis xyz = "0 0 1"/>
+        <limit effort = "1.0" velocity = "5.0" lower ="-3.14" upper = "3.14" />
+        <dynamics damping = "0.2"/>
+    </joint>
+    <link name="rear_left_caster">
+        <visual>
+            <origin xyz="0 0 0" rpy="1.5708 0 0"/>
+            <geometry>
+                <cylinder radius="0.0762" length="0.0508"/>
+            </geometry>
+        </visual>
+        <collision>
+            <origin xyz="0 0 0" rpy="1.5708 0 0"/>
+            <geometry>
+                <cylinder radius="0.0762" length="0.0508"/>
+            </geometry>
+        </collision>
+        <inertial>
+            <mass value="0.5"/>
+            <origin xyz="0 0 0" rpy="0 0 0"/>
+            <inertia ixx="0.001" iyy="0.001" izz="0.001" ixy="0.0" ixz="0.0" iyz="0.0"/>
+        </inertial>
+    </link>
+    <!--Friction for Rear Left Caster-->
+    <gazebo reference="rear_left_caster">
+        <mu1>0.1</mu1>
+        <mu2>0.1</mu2>
+    </gazebo>
+    <!--Reat right caster-->
+    <joint name="rear_right_caster_joint" type="revolute">
+        <parent link="base_link"/>
+        <child link="rear_right_caster"/>
+        <origin xyz="-0.4699 -0.24765 0.0762" rpy="0 0 0"/>
+        <axis xyz = "0 0 1"/>
+        <limit effort = "1.0" velocity = "5.0" lower ="-3.14" upper = "3.14" />
+        <dynamics damping = "0.2"/>
+    </joint>
+    <link name="rear_right_caster">
+        <visual>
+            <origin xyz="0 0 0" rpy="1.5708 0 0"/>
+            <geometry>
+                <cylinder radius="0.0762" length="0.0508"/>
+            </geometry>
+        </visual>
+        <collision>
+            <origin xyz="0 0 0" rpy="1.5708 0 0"/>
+            <geometry>
+                <cylinder radius="0.0762" length="0.0508"/>
+            </geometry>
+        </collision>
+        <inertial>
+            <mass value="0.5"/>
+            <origin xyz="0 0 0" rpy="0 0 0"/>
+            <inertia ixx="0.001" iyy="0.001" izz="0.001" ixy="0.0" ixz="0.0" iyz="0.0"/>
+        </inertial>
+    </link>
+    <!--Friction for rear Right Caster-->
+    <gazebo reference="rear_right_caster">
+        <mu1>0.1</mu1>
+        <mu2>0.1</mu2>
+    </gazebo>
+    <!--Chair-->
     <joint name="chair_joint" type="fixed">
         <parent link="base_link"/>
         <child link="chair"/>
-        <origin rpy="0 0 0" xyz="0 0 0.381"/>
+        <origin rpy="0 0 0" xyz="0 0 0.5334"/>
     </joint>
     <link name="chair">
@@ -88,5 +255,5 @@
             <origin rpy="0 0 0" xyz="0 0 0.3556"/>
             <geometry>
-                <box size="0.4826 0.508 0.7112"/>
+                <box size="0.508 0.4826 0.7112"/>
             </geometry>
         </visual>
@@ -94,5 +261,5 @@
             <origin rpy="0 0 0" xyz="0 0 0.3556"/>
             <geometry>
-                <box size="0.4826 0.508 0.7112"/>
+                <box size="0.508 0.4826 0.7112"/>
             </geometry>
         </collision>
@@ -101,7 +268,8 @@
             <mass value="10.0"/>
             <origin xyz="0 0 0.3556" rpy="0 0 0"/>
-            <inertia ixx="0.3" ixy="0.0" ixz="0.0" iyy="0.3" iyz="0.0" izz="0.3"/>
-        </inertial>
-    </link>
+            <inertia ixx="0.5" ixy="0.0" ixz="0.0" iyy="0.5" iyz="0.0" izz="0.5"/>
+        </inertial>
+    </link>
+    <!--Differential Drive-->
     <gazebo>
         <plugin name="diff_drive_controller" filename="libgazebo_ros_diff_drive.so">
@@ -115,6 +283,7 @@
             <right_joint>right_wheel_joint</right_joint>
             <!-- Physical params -->
-            <wheel_separation>0.5588</wheel_separation>  <!-- distance between wheels -->
-            <wheel_radius>0.3175</wheel_radius>          <!-- radius of your wheel -->
+            <wheel_separation>0.4953</wheel_separation>  <!-- distance between wheels -->
+            <wheel_radius>0.15875</wheel_radius>          <!-- radius of wheel -->
+            <wheel_diameter>0.3175</wheel_diameter>         <!--Wheel diameter-->
             <!-- Odometry settings -->
             <publish_odom>true</publish_odom>
@@ -125,6 +294,7 @@
             <update_rate>50</update_rate>
             <cmd_vel_topic>/cmd_vel</cmd_vel_topic>
-            <max_wheel_torque>10.0</max_wheel_torque>
+            <max_wheel_torque>200.0</max_wheel_torque>
         </plugin>
     </gazebo>
+    <xacro:include filename="$(find robot_sim)/urdf/depth_camera.xacro" />
 </robot>

Commit message: fixed wheel position, wheel traction, caster position, center of mass

File: src/robot_sim/urdf/watcher.urdf.xacro (robot description, xacro)
@@ -26,5 +26,5 @@
         <inertial>
             <mass value="30.0"/>
-            <origin xyz="0 0 0.1778" rpy="0 0 0"/>
+            <origin xyz="0 0 0.1" rpy="0 0 0"/>
             <inertia ixx="1.0" ixy="0.0" ixz="0.0" iyy="1.0" iyz="0.0" izz="1.0"/>
         </inertial>
@@ -35,5 +35,6 @@
         <child link="right_wheel"/>
         <axis xyz="0 1 0"/>
-        <origin rpy="0 0 0" xyz="0 0.24765 0.15875"/>
+        <origin rpy="0 0 0" xyz="0 0.24765 0.13"/><!--changed Z from 0.15875 & again from 0.127-->
+        <dynamics damping="0.5" friction="0.0"/>
     </joint>
     <link name="right_wheel">
@@ -77,5 +78,6 @@
         <child link="left_wheel"/>
         <axis xyz="0 1 0"/>
-        <origin rpy="0 0 0" xyz="0 -0.24765 0.15875"/>
+        <origin rpy="0 0 0" xyz="0 -0.24765 0.127"/>
+        <dynamics damping="0.5" friction="0.0"/>
     </joint>
     <link name="left_wheel">
@@ -119,5 +121,5 @@
         <parent link="base_link"/>
         <child link="front_left_caster"/>
-        <origin xyz="0.3429 0.24765 0.0762" rpy="0 0 0"/>
+        <origin xyz="0.3426 0.26265 0.05" rpy="0 0 0"/>
         <axis  xyz = "0 0 1"/>
         <limit effort = "1.0" velocity = "5.0" lower ="-3.14" upper = "3.14" />
@@ -145,6 +147,6 @@
     <!--Friction for Left Caster wheel-->
     <gazebo reference="front_left_caster">
-        <mu1>0.01</mu1>
-        <mu2>0.01</mu2>
+        <mu1>0.001</mu1>
+        <mu2>0.001</mu2>
     </gazebo>
     <!--Front Right Caster Wheel-->
@@ -152,5 +154,5 @@
         <parent link="base_link"/>
         <child link="front_right_caster"/>
-        <origin xyz="0.3429 -0.24765 0.0762" rpy="0 0 0"/>
+        <origin xyz="0.3426 -0.26265 0.05" rpy="0 0 0"/>
         <axis xyz = "0 0 1"/>
         <limit effort = "1.0" velocity = "5.0" lower ="-3.14" upper = "3.14" />
@@ -178,6 +180,6 @@
     <!--Friction for front right Caster-->
     <gazebo reference="front_right_caster">
-        <mu1>0.1</mu1>
-        <mu2>0.1</mu2>
+        <mu1>0.001</mu1>
+        <mu2>0.001</mu2>
     </gazebo>
     <!--Rear Left  Caster Wheel-->
@@ -185,5 +187,5 @@
         <parent link="base_link"/>
         <child link="rear_left_caster"/>
-        <origin xyz="-0.4699 0.24765 0.0762" rpy="0 0 0"/>
+        <origin xyz="-0.4699 0.24765 0.05" rpy="0 0 0"/>
         <axis xyz = "0 0 1"/>
         <limit effort = "1.0" velocity = "5.0" lower ="-3.14" upper = "3.14" />
@@ -211,6 +213,6 @@
     <!--Friction for Rear Left Caster-->
     <gazebo reference="rear_left_caster">
-        <mu1>0.1</mu1>
-        <mu2>0.1</mu2>
+        <mu1>0.001</mu1>
+        <mu2>0.001</mu2>
     </gazebo>
     <!--Reat right caster-->
@@ -218,5 +220,5 @@
         <parent link="base_link"/>
         <child link="rear_right_caster"/>
-        <origin xyz="-0.4699 -0.24765 0.0762" rpy="0 0 0"/>
+        <origin xyz="-0.4699 -0.24765 0.05" rpy="0 0 0"/>
         <axis xyz = "0 0 1"/>
         <limit effort = "1.0" velocity = "5.0" lower ="-3.14" upper = "3.14" />
@@ -244,6 +246,6 @@
     <!--Friction for rear Right Caster-->
     <gazebo reference="rear_right_caster">
-        <mu1>0.1</mu1>
-        <mu2>0.1</mu2>
+        <mu1>0.001</mu1>
+        <mu2>0.001</mu2>
     </gazebo>
     <!--Chair-->
