Commit message: fixed camera, and camera position on chair

File: src/robot_sim/urdf/depth_camera.xacro (robot description, xacro)
@@ -1,59 +1,65 @@
 <?xml version="1.0"?>
-<robot xmlns:xacro = "http://wwww.ros.org/wiki/xacro">
- <!--CAMERA JOINT -->
-    <joint name = "depth_camera_joint" type = "fixed">
-        <parent link = "base_link"/>
-        <child link = "depth_camera_link"/>
-        <origin xyz = "0.0 0 0.3" rpy = "0 0 0"/>
+<robot xmlns:xacro="http://www.ros.org/wiki/xacro">
+  <xacro:macro name="depth_camera" params="parent">
+    <!-- Camera Joint -->
+    <joint name="depth_camera_joint" type="fixed">
+      <!-- <parent link="${parent}"/> -->
+      <parent link="base_footprint"/>
+      <child link="depth_camera_link"/>
+      <origin xyz="0 0 1.3" rpy="0 0 0"/>
     </joint>
-    <!--Camera LINK-->
-    <link name = "depth_camera_link">
-        <visual>
-            <origin xyz = "0 0 0" rpy = "0 0 0"/>
-            <geometry>
-                <box size ="0.05 0.05 0.05"/>
-            </geometry>
-            <material>
-                <color rgba = "0.2 0.2 0.2 1.0"/>
-            </material>
-        </visual>
-        <collision>
-            <origin xyz="0 0 0" rpy="0 0 0"/>
-            <geometry>
-                <box size="0.05 0.05 0.05"/>
-            </geometry>
-        </collision>
-        <inertial>
-            <mass value="0.01"/>
-            <origin xyz="0 0 0" rpy="0 0 0"/>
-            <inertia ixx="0.00001" iyy="0.00001" izz="0.00001" ixy="0.0" ixz="0.0" iyz="0.0"/>
-        </inertial>
-        <sensor name="depth_camera" type="depth">
-            <pose> 0 0 0 0 0 0 </pose>
-            <always_on>true</always_on>
-            <update_rate>30</update_rate>
-            <visualize>true</visualize>
+    <!-- Camera Link -->
+    <link name="depth_camera_link">
+      <visual>
+        <origin xyz="0 0 0" rpy="0 0 0"/>
+        <geometry>
+          <box size="0.05 0.05 0.05"/>
+        </geometry>
+        <material name = "red">
+          <color rgba="1.0 0.0 0.0 1.0"/>
+        </material>
+      </visual>
+      <collision>
+        <origin xyz="0 0 0" rpy="0 0 0"/>
+        <geometry>
+          <box size="0.05 0.05 0.05"/>
+        </geometry>
+      </collision>
+      <inertial>
+        <mass value="0.01"/>
+        <origin xyz="0 0 0" rpy="0 0 0"/>
+        <inertia ixx="0.00001" iyy="0.00001" izz="0.00001" ixy="0.0" ixz="0.0" iyz="0.0"/>
+      </inertial>
+    </link>
+    <!--Sensor placed correctly inside link -->
+    <gazebo reference="depth_camera_link">
+      <sensor name="depth_camera" type="depth">
+        <pose>0 0 0 0 0 0</pose>
+        <always_on>true</always_on>
+        <update_rate>30</update_rate>
+        <visualize>true</visualize>
         <camera>
-            <horizontal_fov>1.047</horizontal_fov> <!-- ~60 degrees -->
-            <image>
-                <width>640</width>
-                <height>480</height>
-                <format>R8G8B8</format>
-            </image>
-        <clip>
+          <horizontal_fov>1.047</horizontal_fov>
+          <image>
+            <width>640</width>
+            <height>480</height>
+            <format>R8G8B8</format>
+          </image>
+          <clip>
             <near>0.1</near>
             <far>10.0</far>
-        </clip>
+          </clip>
         </camera>
-        <plugin name="gazebo_ros_depth_camera" filename="libgazebo_ros_depth_camera.so">
-            <ros>
-                <namespace>/depth_camera</namespace>
-            </ros>
-            <image_topic_name>image_raw</image_topic_name>
-            <depth_image_topic_name>depth/image_raw</depth_image_topic_name>
-            <camera_info_topic_name>camera_info</camera_info_topic_name>
-            <frame_name>depth_camera_link</frame_name>
+        <plugin name="depth_camera_controller" filename="libgazebo_ros_camera.so">
+          <ros>
+            <namespace>/depth_camera</namespace>
+          </ros>
+          <image_topic_name>image_raw</image_topic_name>
+          <depth_image_topic_name>depth/image_raw</depth_image_topic_name>
+          <camera_info_topic_name>camera_info</camera_info_topic_name>
+          <frame_name>depth_camera_link</frame_name>
         </plugin>
-        </sensor>
-    </link>
+      </sensor>
+    </gazebo>
+  </xacro:macro>
 </robot>

File: src/robot_sim/urdf/watcher.urdf.xacro (robot description, xacro)
@@ -1,4 +1,6 @@
 <?xml version="1.0"?>
 <robot xmlns:xacro="http://www.ros.org/wiki/xacro" name="Watcher">
+    <xacro:include filename="$(find robot_sim)/urdf/depth_camera.xacro" />
+    <!-- <xacro:include filename ="depth_camera.xacro"> -->
     <link name="base_footprint"/>
     <joint name="base_joint" type="fixed">
@@ -297,4 +299,4 @@
         </plugin>
     </gazebo>
-    <xacro:include filename="$(find robot_sim)/urdf/depth_camera.xacro" />
+    <xacro:depth_camera parent="chair"/>
 </robot>

Commit message: Camera height

File: src/robot_sim/urdf/depth_camera.xacro (robot description, xacro)
@@ -7,5 +7,5 @@
       <parent link="base_footprint"/>
       <child link="depth_camera_link"/>
-      <origin xyz="0 0 1.3" rpy="0 0 0"/>
+      <origin xyz="0 0 1.5" rpy="0 0 0"/>
     </joint>
     <!-- Camera Link -->

Commit message: Added lidar sensor

File: src/robot_sim/urdf/depth_camera.xacro (robot description, xacro)
@@ -23,5 +23,5 @@
         <origin xyz="0 0 0" rpy="0 0 0"/>
         <geometry>
-          <box size="0.05 0.05 0.05"/>
+          <box size="0.1245 0.0265 0.0305"/>
         </geometry>
       </collision>

File: src/robot_sim/urdf/watcher.urdf.xacro (robot description, xacro)
@@ -2,4 +2,5 @@
 <robot xmlns:xacro="http://www.ros.org/wiki/xacro" name="Watcher">
     <xacro:include filename="$(find robot_sim)/urdf/depth_camera.xacro" />
+    <xacro:include filename="$(find robot_sim)/urdf/lidar.xacro" />
     <!-- <xacro:include filename ="depth_camera.xacro"> -->
     <link name="base_footprint"/>
@@ -302,3 +303,4 @@
     </gazebo>
     <xacro:depth_camera parent="chair"/>
+    <xacro:lidar_sensor parent="chair" />
 </robot>
